File: BOOST_package/KiCad/BOOST_control_RC2.kicad_pcb (KiCad board)
At the start: 6 copper layers, 45 x 45 mm, 168 parts, among them J11 Conn_02x15_2.54mm, J9 Conn_01x11, Q1 PNP, U101 74HC00, U102 74HC00, U103 74HC00, U104 74HC14, U105 74HC14, U106 CD74HC4066, U13 TLV9001, U14 MCP6561, U18 4017, U2 MCP6561, U21 MCP6561, U22 TLV9001, U23 TLV9001, U24 TLV9001, U26 MCP4451-103E/ST, U28 74HC4051, U3 TLV9001, U4 MCP6561, U5 MCP6561, U7 TLV9001

Commit message: going to send out
Parts:
- added R106: 4.7k, Resistor_SMD:R_0603_1608Metric, F.Cu at (57.1, 94.0)
- added R107: 4.7k, Resistor_SMD:R_0603_1608Metric, F.Cu at (55.1, 101.5)
- D1, D15, D20, D24, D27, D3, D4, D5, D6, D7: value D -> 1N4148W
- D23, D25, D26: value D -> BAT54WS
- R102, R99: value 10k -> 1k
Connections:
- net Net-(U102B-A) renamed OUT_1_ENA
- net Net-(U102C-A) renamed OUT_2_ENA
- net Net-(U103A-A) renamed OUT_3_ENA
- net Net-(U18-Q3) renamed 4
Routing:
- net SDA: track 22.7 -> 27.9 mm, vias 1 -> 2
- net Net-(D5--): track 41.0 -> 46.1 mm, vias 4 -> 5
- net 5V: track 42.7 -> 40.7 mm, vias 35 -> 36
- net SCL: track 9.42 -> 10.7 mm
- net Net-(U101A-Y): track 17.2 -> 16.4 mm
- net GND: vias 72 -> 74
