File: BOOST_package/KiCad/BOOST.kicad_sch (KiCad schematic)
At the start: 293 parts, among them J1 Conn_01x01_Pin, J10 Conn_02x15_2.54mm, J11 Conn_02x15_2.54mm, J2 Conn_01x01_Pin, J3 Conn_01x01_Pin, J4 Conn_01x01_Pin, J5 Conn_01x01_Pin, J6 Conn_01x01_Pin, J7 Conn_01x01_Pin, J8 Conn_01x01_Pin, J9 Conn_01x11, M1 HYG180N10, M10 HYG180N10, M2 HYG180N10, M3 HYG180N10, M4 HYG180N10, M5 HYG180N10, M6 HYG180N10, M7 HYG180N10, M8 HYG180N10, M9 HYG180N10, Q1 PNP, U1 L78L05_SOT89, U10 UCC21520DW, U101 74HC00, U102 74HC00, U103 74HC00, U104 74HC14, U105 74HC14, U106 CD74HC4066, U11 TLV9001, U12 TLV9001, U13 TLV9001, U14 MCP6561, U15 UCC21520DW, U16 MC7812, U17 L78L05_SOT89, U18 4017, U19 UCC21520DW, U2 MCP6561, U21 MCP6561, U22 TLV9001, U23 TLV9001, U24 TLV9001, U25 INA241A4xD, U26 MCP4451-103E/ST, U28 74HC4051, U3 TLV9001, U4 MCP6561, U5 MCP6561, U6 TLV9001, U7 TLV9001, U8 UCC21520DW

Commit message: going to send out
Parts:
- removed R14: 1Meg, Resistor_SMD:R_0805_2012Metric, symbol ltspice:res
- added R106, R107: 4.7k, Resistor_SMD:R_0603_1608Metric, symbol ltspice:res
- D1, D15, D20, D24, D27, D3, D4, D5, D6, D7: value D -> 1N4148W
- D10, D21, D9: value D -> BAV21W
- D11, D13, D14, D2, D22, D8: value D -> B5819W
- D23, D25, D26: value D -> BAT54WS
- J1: value Conn_01x01_Pin -> Vin+
- J2: value Conn_01x01_Pin -> Vin-
- J3: value Conn_01x01_Pin -> Out1+
- J4: value Conn_01x01_Pin -> Out1-
- J5: value Conn_01x01_Pin -> Out3+
- J6: value Conn_01x01_Pin -> Out3-
- J7: value Conn_01x01_Pin -> Out2-
- J8: value Conn_01x01_Pin -> Out2+
- R102, R99: value 10k -> 1k
Connections:
- net 5V: now also R106.1, R107.1
- net SCL: now also R106.2
- net SDA: now also R107.2
- net OUT_1_ENA: now reaches U102.4 (A), U18.3 (Q0), U28.11 (S0)
- net OUT_2_ENA: now reaches U102.10 (A), U18.2 (Q1), U28.10 (S1)
- net OUT_3_ENA: now reaches U103.1 (A), U18.4 (Q2), U28.9 (S2)
- net 4: now reaches U18.15 (Reset), U18.7 (Q3)
Other:
- note added: "0-5V PWM signal sent from arduino to control brightness"
- note added: "0-5V PWM to set minimum voltage reference This will be connected to an arduino pin"
- note added: "1 mOhm shunt: measures inductor current"
- note added: "CH1 HEADROOM SERVO"
- note added: "CH1 LED CURRENT LIMIT"
- note added: "CH2 HEADROOM SERVO"
- note added: "CH2 LED CURRENT LIMIT"
- note added: "CH3 HEADROOM SERVO"
- note added: "CH3 LED CURRENT LIMIT"
- note added: "CHANNEL ENABLE"
- note added: "CONNECTORS"
- note added: "Channel 1 output-voltage error amplifier, Vout_1 -> Verr1"
- note added: "Channel 2 output-voltage error amplifier, Vout_2 -> Verr2"
- note added: "Channel 3 output-voltage error amplifier, Vout_3 -> Verr3"
- note added: "D28-D30: pre-charge diodes Vin -> Vout_1/2/3"
- note added: "I added a lot of capacitors for individual components in the kicad, which are all put here"
- note added: "I2C pull-ups (U26 has none)"
- note added: "LOW-ERROR TIMEOUT"
- note added: "M1 INHIBIT"
- note added: "M1 ON/OFF LATCH"
- note added: "OUTPUT 1"
- note added: "OUTPUT 2"
- note added: "OUTPUT 3"
- note added: "SEQUENCER / ERROR SELECT"
- note added: "Signal that can be sent from the arduino to disable the circuit"
- note added: "U26A: one of the 4 pots inside U26 (MCP4451)"
- note added: "U26B: one of the 4 pots inside U26 (MCP4451)"
- note added: "U26C: one of the 4 pots inside U26 (MCP4451)"
- note added: "U26E: MCP4451 control unit, serves U26A/B/C"
- note added: "actual led diode will not be on the pcb"
- note added: "bootstrap capacitors"
- note added: "clamps LX spikes"
- note added: "connects LX to output 1"
- note added: "connects LX to output 2"
- note added: "connects LX to output 3"
- note added: "current sense amplifies R1 voltage by 100x"
- note added: "digital potentiometer to control current"
- note added: "disables m1 if there is 0 error on the current channel"
- note added: "error signal - used to control how long the inductor charges up for"
- note added: "filters the PWM to DC"
- note added: "gate driver"
- note added: "goes to gate driver"
- note added: "inhibits m1 if 12V rail is below 9.8V"
- note added: "logic chip supply pins"
- note added: "low side switch"
- note added: "makes it so that if there is one channel with low error, it doesn't just stop on that one channel."
- note added: "mosfet used as a kind of variable resistor to keep led current from going too high."
- note added: "op amp will try to make its output match the reference current"
- note added: "rc circuit delays m1 turn on diode creates fast turn off"
- note added: "same as channel 1"
- note added: "spare units (not used)"
- note added: "switch used so that circuit only samples while the led is on"
- note added: "this pushes up the reference voltage if the output voltage is undershooting for a long time"
- note added: "when m1 pulls inductor to ground, current can conduct through the mosfet body diode to charge up this capacitor"
- title: (none) -> BOOST LED driver - main schematic (both boards)
- moved on the sheet: C1, C10, C100, C101, C102, C103, C104, C11, C12, C13, C14, C15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
