File: BOOST_package/KiCad/BOOST_power_RC2.kicad_pcb (KiCad board)
At the start: 6 copper layers, 74 x 86 mm, 135 parts, among them J1 Conn_01x01_Pin, J10 Conn_02x15_2.54mm, J2 Conn_01x01_Pin, J3 Conn_01x01_Pin, J4 Conn_01x01_Pin, J5 Conn_01x01_Pin, J6 Conn_01x01_Pin, J7 Conn_01x01_Pin, J8 Conn_01x01_Pin, M1 HYG180N10, M10 HYG180N10, M2 HYG180N10, M3 HYG180N10, M4 HYG180N10, M5 HYG180N10, M6 HYG180N10, M7 HYG180N10, M8 HYG180N10, M9 HYG180N10, U1 L78L05_SOT89, U10 UCC21520DW, U11 TLV9001, U12 TLV9001, U15 UCC21520DW, U16 MC7812, U17 L78L05_SOT89, U19 UCC21520DW, U25 INA241A4xD, U6 TLV9001, U8 UCC21520DW

Commit message: going to send out
Parts:
- removed R14: 1Meg, Resistor_SMD:R_0805_2012Metric
- D10, D21, D9: value D -> BAV21W
- D11, D13, D14, D2, D22, D8: value D -> B5819W
- J1: value Conn_01x01_Pin -> Vin+
- J2: value Conn_01x01_Pin -> Vin-
- J3: value Conn_01x01_Pin -> Out1+
- J4: value Conn_01x01_Pin -> Out1-
- J5: value Conn_01x01_Pin -> Out3+
- J6: value Conn_01x01_Pin -> Out3-
- J7: value Conn_01x01_Pin -> Out2-
- J8: value Conn_01x01_Pin -> Out2+
Routing:
- net 12V: track 129.4 -> 110.6 mm, vias 12 -> 9
- net LX: track 2.95 -> 0.00 mm, vias 114 -> 112
- net Vout_3: vias 78 -> 80
- net Vin: vias 143 -> 142
- net GND: vias 277 -> 279
