File: BOOST_split_boards/previous/2026-09-28/before_reorganized_schematics/BOOST.kicad_sch (KiCad schematic)
At the start: 290 parts, among them J1 Conn_01x01_Pin, J10 Conn_02x15_2.54mm, J11 Conn_02x15_2.54mm, J2 Conn_01x01_Pin, J3 Conn_01x01_Pin, J4 Conn_01x01_Pin, J5 Conn_01x01_Pin, J6 Conn_01x01_Pin, J7 Conn_01x01_Pin, J8 Conn_01x01_Pin, J9 Conn_01x11, M1 HYG180N10, M10 HYG180N10, M2 HYG180N10, M3 HYG180N10, M4 HYG180N10, M5 HYG180N10, M6 HYG180N10, M7 HYG180N10, M8 HYG180N10, M9 HYG180N10, Q1 PNP, U1 L78L05_SOT89, U10 UCC21520DW, U101 74HC00, U102 74HC00, U103 74HC00, U104 74HC14, U105 74HC14, U106 CD74HC4066, U11 MCP6241, U12 MCP6241, U13 MCP6241, U14 MCP6561, U15 UCC21520DW, U16 LM2940_12, U17 L78L05_SOT89, U18 4017, U19 UCC21520DW, U2 MCP6561, U21 MCP6561, U22 MCP6241, U23 MCP6241, U24 MCP6241, U25 INA241A4xD, U26 MCP4451-103E/ST, U28 74HC4051, U3 MCP6241, U4 MCP6561, U5 MCP6561, U6 MCP6241, U7 MCP6241, U8 UCC21520DW

Commit message: added diodes from input to output
Other:
- moved on the sheet: C41, C44, C45, D27, R105
