File: BOOST_schematic_cleanup/KiCad/BOOST_control_RC2.kicad_pcb (KiCad board)
At the start: 8 copper layers, 45 x 45 mm, 168 parts, among them J11 Conn_02x15_2.54mm, J9 Conn_01x11, Q1 PNP, U101 74HC00, U102 74HC00, U103 74HC00, U104 74HC14, U105 74HC14, U106 CD74HC4066, U13 MCP6241, U14 MCP6561, U18 4017, U2 MCP6561, U21 MCP6561, U22 MCP6241, U23 MCP6241, U24 MCP6241, U26 MCP4451-103E/ST, U28 74HC4051, U3 MCP6241, U4 MCP6561, U5 MCP6561, U7 MCP6241

Commit message: changed power board to 6 layers
Parts:
- U13, U22, U23, U24, U3, U7: value MCP6241 -> TLV9001
Routing:
- added copper zone on In2.Cu, net 5V
- added copper zone on In3.Cu, net GND
- removed copper zone on In3.Cu, net 5V
- removed copper zone on In2.Cu, net GND
- removed copper zone on In5.Cu, net GND
- removed copper zone on In6.Cu, net GND
Other:
- copper layers 8 -> 6
